Commit message: cambios

File: src/dif_bot_description/urdf/dif_bot_properties.xacro (robot description, xacro)
@@ -1,95 +1,14 @@
 <?xml version="1.0"?>
-<robot xmlns:xacro="http://www.ros.org/wiki/xacro" name="dif_bot">
-  <!-- Definición de colores materiales -->
-  <material name="blue">
-    <color rgba="0.0 0.0 0.8 1.0"/>
-  </material>
-  <material name="black">
-    <color rgba="0.1 0.1 0.1 1.0"/>
-  </material>
-  <material name="white">
-    <color rgba="1.0 1.0 1.0 1.0"/>
-  </material>
-  <!-- Base Link (Huella virtual en el suelo) -->
-  <link name="base_link"/>
-  <!-- Chasis del Robot -->
-  <joint name="base_joint" type="fixed">
-    <parent link="base_link"/>
-    <child link="chassis"/>
-    <origin xyz="0 0 0.1" rpy="0 0 0"/>
-  </joint>
-  <link name="chassis">
-    <visual>
-      <origin xyz="0 0 0" rpy="0 0 0"/>
-      <geometry>
-        <box size="0.5 0.3 0.1"/>
-      </geometry>
-      <material name="blue"/>
-    </visual>
-    <collision>
-      <origin xyz="0 0 0" rpy="0 0 0"/>
-      <geometry>
-        <box size="0.5 0.3 0.1"/>
-      </geometry>
-    </collision>
-  </link>
-  <!-- Rueda Izquierda -->
-  <joint name="left_wheel_joint" type="continuous">
-    <parent link="chassis"/>
-    <child link="left_wheel"/>
-    <origin xyz="0.1 0.175 -0.05" rpy="-1.5707 0 0"/>
-    <axis xyz="0 0 1"/>
-  </joint>
-  <link name="left_wheel">
-    <visual>
-      <geometry>
-        <cylinder radius="0.05" length="0.04"/>
-      </geometry>
-      <material name="black"/>
-    </visual>
-    <collision>
-      <geometry>
-        <cylinder radius="0.05" length="0.04"/>
-      </geometry>
-    </collision>
-  </link>
-  <!-- Rueda Derecha -->
-  <joint name="right_wheel_joint" type="continuous">
-    <parent link="chassis"/>
-    <child link="right_wheel"/>
-    <origin xyz="0.1 -0.175 -0.05" rpy="-1.5707 0 0"/>
-    <axis xyz="0 0 1"/>
-  </joint>
-  <link name="right_wheel">
-    <visual>
-      <geometry>
-        <cylinder radius="0.05" length="0.04"/>
-      </geometry>
-      <material name="black"/>
-    </visual>
-    <collision>
-      <geometry>
-        <cylinder radius="0.05" length="0.04"/>
-      </geometry>
-    </collision>
-  </link>
-  <!-- Rueda Loca (Caster Wheel) -->
-  <joint name="caster_wheel_joint" type="fixed">
-    <parent link="chassis"/>
-    <child link="caster_wheel"/>
-    <origin xyz="-0.15 0 -0.075" rpy="0 0 0"/>
-  </joint>
-  <link name="caster_wheel">
-    <visual>
-      <geometry>
-        <sphere radius="0.025"/>
-      </geometry>
-      <material name="white"/>
-    </visual>
-    <collision>
-      <geometry>
-        <sphere radius="0.025"/>
-      </geometry>
-    </collision>
-  </link>
+<robot xmlns:xacro="http://www.ros.org/wiki/xacro">
+  <!-- Propiedades del Chasis -->
+  <xacro:property name="chassis_length" value="0.5"/>
+  <xacro:property name="chassis_width" value="0.3"/>
+  <xacro:property name="chassis_height" value="0.1"/>
+  <!-- Propiedades de las Ruedas -->
+  <xacro:property name="wheel_radius" value="0.05"/>
+  <xacro:property name="wheel_length" value="0.04"/>
+  <xacro:property name="wheel_ygap" value="0.175"/>
+  <xacro:property name="wheel_zoff" value="-0.05"/>
+  <!-- Propiedad de la Rueda Loca -->
+  <xacro:property name="caster_radius" value="0.025"/>
 </robot>
