Commit message: cambios

File: src/dif_bot_description/urdf/dif_bot.urdf.xacro (robot description, xacro)
@@ -1,5 +1,5 @@
 <?xml version="1.0"?>
 <robot xmlns:xacro="http://www.ros.org/wiki/xacro" name="dif_bot">
-  <!-- Importar archivo de propiedades (debe ir primero) -->
+  <!-- Importar propiedades -->
   <xacro:include filename="$(find dif_bot_description)/urdf/dif_bot_properties.xacro"/>
   <!-- Materiales -->
@@ -13,4 +13,32 @@
     <color rgba="1.0 1.0 1.0 1.0"/>
   </material>
+  <!-- ==================== MACROS DE INERCIA ==================== -->
+  <xacro:macro name="box_inertia" params="m w h d">
+    <inertial>
+      <origin xyz="0 0 0" rpy="0 0 0"/>
+      <mass value="${m}"/>
+      <inertia ixx="${(m/12) * (h*h + d*d)}" ixy="0.0" ixz="0.0"
+               iyy="${(m/12) * (w*w + d*d)}" iyz="0.0"
+               izz="${(m/12) * (w*w + h*h)}"/>
+    </inertial>
+  </xacro:macro>
+  <xacro:macro name="cylinder_inertia" params="m r h">
+    <inertial>
+      <origin xyz="0 0 0" rpy="0 0 0"/>
+      <mass value="${m}"/>
+      <inertia ixx="${(m/12) * (3*r*r + h*h)}" ixy="0.0" ixz="0.0"
+               iyy="${(m/12) * (3*r*r + h*h)}" iyz="0.0"
+               izz="${(m/2) * (r*r)}"/>
+    </inertial>
+  </xacro:macro>
+  <xacro:macro name="sphere_inertia" params="m r">
+    <inertial>
+      <origin xyz="0 0 0" rpy="0 0 0"/>
+      <mass value="${m}"/>
+      <inertia ixx="${(2.0/5.0) * m * (r*r)}" ixy="0.0" ixz="0.0"
+               iyy="${(2.0/5.0) * m * (r*r)}" iyz="0.0"
+               izz="${(2.0/5.0) * m * (r*r)}"/>
+    </inertial>
+  </xacro:macro>
   <!-- Base Footprint -->
   <link name="base_footprint"/>
@@ -42,4 +70,5 @@
       </geometry>
     </collision>
+    <xacro:box_inertia m="${chassis_mass}" w="${chassis_length}" h="${chassis_width}" d="${chassis_height}"/>
   </link>
   <!-- Macro para las ruedas -->
@@ -63,4 +92,5 @@
         </geometry>
       </collision>
+      <xacro:cylinder_inertia m="${wheel_mass}" r="${wheel_radius}" h="${wheel_length}"/>
     </link>
   </xacro:macro>
@@ -86,4 +116,5 @@
       </geometry>
     </collision>
+    <xacro:sphere_inertia m="${caster_mass}" r="${caster_radius}"/>
   </link>
 </robot>

File: src/dif_bot_description/urdf/dif_bot_properties.xacro (robot description, xacro)
@@ -5,4 +5,5 @@
   <xacro:property name="chassis_width" value="0.3"/>
   <xacro:property name="chassis_height" value="0.1"/>
+  <xacro:property name="chassis_mass" value="1.0"/>
   <!-- Propiedades de las Ruedas -->
   <xacro:property name="wheel_radius" value="0.05"/>
@@ -10,5 +11,7 @@
   <xacro:property name="wheel_ygap" value="0.175"/>
   <xacro:property name="wheel_zoff" value="-0.05"/>
+  <xacro:property name="wheel_mass" value="0.1"/>
   <!-- Propiedad de la Rueda Loca -->
   <xacro:property name="caster_radius" value="0.025"/>
+  <xacro:property name="caster_mass" value="0.05"/>
 </robot>
